Commit message: Updated message files, cleaned up the launch files, updated the rviz config for new topic names. Updated the versioned robot description, parameterized the launch files so folks can pass in their own robot descriptions.

File: description/atlas_unplugged_v5_no_hands.urdf (robot description, URDF)
Before this commit: robot atlas, 47 links, 46 joints
Links:
- removed link l_farm
- removed link r_farm
- removed link rear_situational_awareness_camera_link
- removed link rear_situational_awareness_camera_optical_frame
- added link l_lfarm, mass 0.648; collision cylinder length=0.015 radius=0.045; collision cylinder length=0.015 radius=0.052
- added link l_ufarm, mass 2.4798; collision box size=0.08 0.09 0.11; collision cylinder length=0.1 radius=0.053
- added link r_lfarm, mass 0.648; collision cylinder length=0.015 radius=0.045; collision cylinder length=0.015 radius=0.052
- added link r_ufarm, mass 2.4798; collision box size=0.08 0.09 0.11; collision cylinder length=0.1 radius=0.053
- link l_clav: geometry collision box size=0.1 0.07 0.072; collision cylinder length=0.1525 radius=0.0555
- link l_foot: geometry collision box size=0.1 0.08 0.02; collision box size=0.227 0.133887 0.05
- link l_hand: mass 2.509 -> 0.5839; geometry 
- link l_larm: geometry collision box size=0.025 0.06 0.06; collision box size=0.025 0.155 0.07
- link l_lglut: geometry collision box size=0.0975 0.069 0.103; collision cylinder length=0.060306 radius=0.02009687
- link l_lleg: geometry collision cylinder length=0.40 radius=0.07; visual mesh filename=package://atlas_description/meshes_unplugged/l_lleg.dae
- link l_scap: geometry collision box size=0.02 0.029 0.018; collision box size=0.028 0.090 0.05
- link l_talus: geometry collision cylinder length=0.010059 radius=0.010348; collision cylinder length=0.029542 radius=0.010181
- link l_uarm: geometry collision box size=0.05 0.07 0.15; collision cylinder length=0.11 radius=0.065
- link l_uglut: geometry collision cylinder length=0.078396 radius=0.019096; collision cylinder length=0.080842 radius=0.019841
- link l_uleg: geometry collision box size=0.07 0.038 0.14; collision box size=0.07 0.038 0.15
- link ltorso: geometry visual mesh filename=package://atlas_description/meshes_unplugged/ltorso.dae
- link mtorso: geometry collision cylinder length=0.15 radius=0.02; visual mesh filename=package://atlas_description/meshes_unplugged/mtorso.dae
- link pelvis: geometry collision box size=0.1 0.15 0.2; collision cylinder length=0.05 radius=0.16
- link r_clav: geometry collision box size=0.1 0.07 0.072; collision cylinder length=0.1525 radius=0.0555
- link r_foot: geometry collision box size=0.1 0.08 0.02; collision box size=0.227 0.133887 0.05
- link r_hand: mass 2.509 -> 0.5839; geometry 
- link r_larm: geometry collision box size=0.025 0.06 0.06; collision box size=0.025 0.155 0.07
- link r_lglut: geometry collision box size=0.0975 0.069 0.103; collision cylinder length=0.060306 radius=0.02009687
- link r_lleg: geometry collision cylinder length=0.40 radius=0.07; visual mesh filename=package://atlas_description/meshes_unplugged/r_lleg.dae
- link r_scap: geometry collision box size=0.02 0.029 0.018; collision box size=0.028 0.090 0.05
- link r_talus: geometry collision cylinder length=0.010059 radius=0.010348; collision cylinder length=0.029542 radius=0.010181
- link r_uarm: geometry collision box size=0.05 0.07 0.15; collision cylinder length=0.11 radius=0.065
- link r_uglut: geometry collision cylinder length=0.078396 radius=0.019096; collision cylinder length=0.080842 radius=0.019841
- link r_uleg: geometry collision box size=0.07 0.038 0.14; collision box size=0.07 0.038 0.15
- link utorso: mass 66.907 -> 63.73; geometry collision box size=0.2 0.25 0.01; collision box size=0.456306 0.341719 0.12
Joints:
- removed joint l_arm_shy
- removed joint r_arm_shy
- removed joint rear_situational_awareness_camera_joint
- removed joint rear_situational_awareness_camera_optical_frame_joint
- added joint l_arm_shz: type revolute, parent utorso, child l_clav, origin xyz=0.1406 0.2256 0.4776 rpy=0 0 0, axis 0 0 1, limit lower=-1.5708 upper=0.785398 effort=87 velocity=12
- added joint l_arm_wry2: type revolute, parent l_lfarm, child l_hand, origin xyz=0 0 0 rpy=0 0 0, axis 0 1 0, limit lower=-2.9671 upper=2.9671 effort=25 velocity=10
- added joint r_arm_shz: type revolute, parent utorso, child r_clav, origin xyz=0.1406 -0.2256 0.4776 rpy=0 0 0, axis 0 0 1, limit lower=-0.785398 upper=1.5708 effort=87 velocity=12
- added joint r_arm_wry2: type revolute, parent r_lfarm, child r_hand, origin xyz=0 0 0 rpy=0 0 0, axis 0 1 0, limit lower=-2.9671 upper=2.9671 effort=25 velocity=10
- joint back_bkx: limit lower=-0.698132 upper=0.698132 effort=200 velocity=12 -> lower=-0.523599 upper=0.523599 effort=300 velocity=12; origin xyz=0 0 0.05 rpy=0 -0 0 -> xyz=0 0 0.05 rpy=0 0 0
- joint back_bky: limit lower=-0.610691 upper=0.438427 effort=206.843 velocity=12 -> lower=-0.219388 upper=0.538783 effort=445 velocity=9; origin xyz=0 0 0.16197 rpy=0 -0 0 -> xyz=0 0 0.162 rpy=0 0 0
- joint back_bkz: limit lower=-0.663225 upper=0.663225 effort=124.016 velocity=12 -> lower=-0.663225 upper=0.663225 effort=106 velocity=12; origin xyz=-0.0125 0 0 rpy=0 -0 0 -> xyz=-0.0125 0 0 rpy=0 0 0
- joint l_arm_elx: limit lower=0 upper=2.35619 effort=114 velocity=12 -> lower=0 upper=2.35619 effort=112 velocity=12; origin xyz=0 0.119 0.00921 rpy=0 -0 0 -> xyz=0 0.119 0.0092 rpy=0 0 0
- joint l_arm_ely: limit lower=0 upper=3.14159 effort=114 velocity=12 -> lower=0 upper=3.14159 effort=63 velocity=12; origin xyz=0 0.187 0.016 rpy=0 -0 0 -> xyz=0 0.187 -0.016 rpy=0 0 0
- joint l_arm_shx: limit lower=-1.5708 upper=1.5708 effort=170 velocity=12 -> lower=-1.5708 upper=1.5708 effort=99 velocity=12; origin xyz=0 0.14035 0.19609 rpy=0 -0 0 -> xyz=0 0.11 -0.245 rpy=0 0 0
- joint l_arm_wrx: child l_hand -> l_lfarm; limit lower=-1.1781 upper=1.1781 effort=60 velocity=12 -> lower=-1.7628 upper=1.7628 effort=25 velocity=10; origin xyz=0 0.119 -0.00921 rpy=0 -0 0 -> xyz=0 0 0 rpy=0 0 0; parent l_farm -> l_ufarm
- joint l_arm_wry: child l_farm -> l_ufarm; limit lower=0 upper=3.14159 effort=114 velocity=12 -> lower=-3.011 upper=3.011 effort=25 velocity=10; origin xyz=0 0.187 -0.00921 rpy=0 -0 0 -> xyz=0 0.29955 -0.00921 rpy=0 0 0
- joint l_leg_akx: limit lower=-0.8 upper=0.8 effort=90 velocity=12 -> lower=-0.8 upper=0.8 effort=360 velocity=12; origin xyz=0 0 0 rpy=0 -0 0 -> xyz=0 0 0 rpy=0 0 0
- joint l_leg_aky: limit lower=-1 upper=0.7 effort=700 velocity=12 -> lower=-1 upper=0.7 effort=740 velocity=12; origin xyz=0 0 -0.422 rpy=0 -0 0 -> xyz=0 0 -0.422 rpy=0 0 0
- joint l_leg_hpx: limit lower=-0.523599 upper=0.523599 effort=180 velocity=12 -> lower=-0.523599 upper=0.523599 effort=530 velocity=12; origin xyz=0 0 0 rpy=0 -0 0 -> xyz=0 0 0 rpy=0 0 0
- joint l_leg_hpy: limit lower=-1.72072 upper=0.524821 effort=260 velocity=12 -> lower=-1.61234 upper=0.65764 effort=840 velocity=12; origin xyz=0.05 0 -0.05 rpy=0 -0 0 -> xyz=0.05 0.0225 -0.066 rpy=0 0 0
- joint l_leg_hpz: limit lower=-0.174533 upper=1.22173 effort=110 velocity=12 -> lower=-0.174358 upper=0.786794 effort=275 velocity=12; origin xyz=0 0.089 0 rpy=0 -0 0 -> xyz=0 0.089 0 rpy=0 0 0
- joint l_leg_kny: limit lower=0 upper=2.38569 effort=220 velocity=12 -> lower=0 upper=2.35637 effort=890 velocity=12; origin xyz=-0.05 0 -0.374 rpy=0 -0 0 -> xyz=-0.05 0 -0.374 rpy=0 0 0
- joint l_situational_awareness_camera_joint: origin xyz=0.216409 0.121799 0.406759 rpy=-1.57079633 0 1.30899694 -> xyz=0.155 0.121 0.785 rpy=0 0 1.309
- joint neck_ry: limit lower=-0.602139 upper=1.14494 effort=5 velocity=12 -> lower=-0.602139 upper=1.14319 effort=25 velocity=6.28; origin xyz=0.21672 0 0.53796 rpy=0 -0 0 -> xyz=0.2946 0 0.5765 rpy=0 0 0
- joint r_arm_elx: limit lower=-2.35619 upper=0 effort=114 velocity=12 -> lower=-2.35619 upper=0 effort=112 velocity=12; origin xyz=0 -0.119 0.00921 rpy=0 -0 0 -> xyz=0 -0.119 0.0092 rpy=0 0 0
- joint r_arm_ely: limit lower=0 upper=3.14159 effort=114 velocity=12 -> lower=0 upper=3.14159 effort=63 velocity=12; origin xyz=0 -0.187 0.016 rpy=0 -0 0 -> xyz=0 -0.187 -0.016 rpy=0 0 0
- joint r_arm_shx: limit lower=-1.5708 upper=1.5708 effort=170 velocity=12 -> lower=-1.5708 upper=1.5708 effort=99 velocity=12; origin xyz=0 -0.14035 0.19609 rpy=0 -0 0 -> xyz=0 -0.11 -0.245 rpy=0 0 0
- joint r_arm_wrx: child r_hand -> r_lfarm; limit lower=-1.1781 upper=1.1781 effort=60 velocity=12 -> lower=-1.7628 upper=1.7628 effort=25 velocity=10; origin xyz=0 -0.119 0.00921 rpy=0 -0 0 -> xyz=0 0 0 rpy=0 0 0; parent r_farm -> r_ufarm
- joint r_arm_wry: child r_farm -> r_ufarm; limit lower=0 upper=3.14159 effort=114 velocity=12 -> lower=-3.011 upper=3.011 effort=25 velocity=10; origin xyz=0 -0.187 -0.00921 rpy=0 -0 0 -> xyz=0 -0.29955 -0.00921 rpy=0 0 0
- joint r_leg_akx: limit lower=-0.8 upper=0.8 effort=90 velocity=12 -> lower=-0.8 upper=0.8 effort=360 velocity=12; origin xyz=0 0 0 rpy=0 -0 0 -> xyz=0 0 0 rpy=0 0 0
- joint r_leg_aky: limit lower=-1 upper=0.7 effort=700 velocity=12 -> lower=-1 upper=0.7 effort=740 velocity=12; origin xyz=0 0 -0.422 rpy=0 -0 0 -> xyz=0 0 -0.422 rpy=0 0 0
- joint r_leg_hpx: limit lower=-0.523599 upper=0.523599 effort=180 velocity=12 -> lower=-0.523599 upper=0.523599 effort=530 velocity=12; origin xyz=0 0 0 rpy=0 -0 0 -> xyz=0 0 0 rpy=0 0 0
- joint r_leg_hpy: limit lower=-1.72072 upper=0.524821 effort=260 velocity=12 -> lower=-1.61234 upper=0.65764 effort=840 velocity=12; origin xyz=0.05 0 -0.05 rpy=0 -0 0 -> xyz=0.05 -0.0225 -0.066 rpy=0 0 0
- joint r_leg_hpz: limit lower=-1.22173 upper=0.174533 effort=110 velocity=12 -> lower=-0.786794 upper=0.174358 effort=275 velocity=12; origin xyz=0 -0.089 0 rpy=0 -0 0 -> xyz=0 -0.089 0 rpy=0 0 0
- joint r_leg_kny: limit lower=0 upper=2.38569 effort=220 velocity=12 -> lower=0 upper=2.35637 effort=890 velocity=12; origin xyz=-0.05 0 -0.374 rpy=0 -0 0 -> xyz=-0.05 0 -0.374 rpy=0 0 0
- joint r_situational_awareness_camera_joint: origin xyz=0.216409 -0.121799 0.406759 rpy=1.57079633 0 -1.30899694 -> xyz=0.155 -0.121 0.785 rpy=0 0 -1.309
