Commit message: Cleanup stuff to use v4 instead of v5 for stopgap release

File: ihmc_models/urdf/atlas_unplugged_v4_no_hands_no_wry2.urdf (robot description, URDF)
Before this commit: robot atlas, 47 links, 46 joints
Links:
- removed link l_farm
- removed link r_farm
- added link l_ufarm, mass 3.388; collision box size=0.135 0.1 0.045; collision cylinder length=0.125 radius=0.045
- added link r_ufarm, mass 3.388; collision box size=0.135 0.1 0.045; collision cylinder length=0.125 radius=0.045
- link l_clav: geometry collision box size=0.1 0.07 0.072; collision cylinder length=0.1525 radius=0.0555
- link l_foot: geometry collision box size=0.1 0.08 0.02; collision box size=0.227 0.133887 0.05
- link l_lglut: geometry collision cylinder length=0.060306 radius=0.02009687; collision cylinder length=0.144 radius=0.02
- link l_lleg: geometry collision cylinder length=0.40 radius=0.07; visual mesh filename=package://atlas_description/meshes_unplugged/l_lleg.dae scale=1 1 1
- link l_scap: geometry collision box size=0.02 0.029 0.018; collision box size=0.028 0.090 0.05
- link l_talus: geometry collision cylinder length=0.010059 radius=0.010348; collision cylinder length=0.029542 radius=0.010181
- link l_uarm: geometry collision box size=0.05 0.07 0.15; collision cylinder length=0.11 radius=0.065
- link l_uglut: geometry collision cylinder length=0.078396 radius=0.019096; collision cylinder length=0.080842 radius=0.019841
- link l_uleg: geometry collision box size=0.07 0.038 0.14; collision box size=0.07 0.038 0.15
- link ltorso: geometry visual mesh filename=package://atlas_description/meshes_unplugged/ltorso.dae scale=1 1 1
- link mtorso: geometry collision cylinder length=0.15 radius=0.02; visual mesh filename=package://atlas_description/meshes_unplugged/mtorso.dae scale=1 1 1
- link pelvis: geometry collision box size=0.1 0.15 0.2; collision cylinder length=0.05 radius=0.16
- link r_clav: geometry collision box size=0.1 0.07 0.072; collision cylinder length=0.1525 radius=0.0555
- link r_foot: geometry collision box size=0.1 0.08 0.02; collision box size=0.227 0.133887 0.05
- link r_lglut: geometry collision cylinder length=0.060306 radius=0.02009687; collision cylinder length=0.142 radius=0.02
- link r_lleg: geometry collision cylinder length=0.40 radius=0.07; visual mesh filename=package://atlas_description/meshes_unplugged/r_lleg.dae scale=1 1 1
- link r_scap: geometry collision box size=0.02 0.029 0.018; collision box size=0.028 0.090 0.05
- link r_talus: geometry collision cylinder length=0.010059 radius=0.010348; collision cylinder length=0.029542 radius=0.010181
- link r_uarm: geometry collision box size=0.05 0.07 0.15; collision cylinder length=0.11 radius=0.065
- link r_uglut: geometry collision cylinder length=0.078396 radius=0.019096; collision cylinder length=0.080842 radius=0.019841
- link r_uleg: geometry collision box size=0.07 0.038 0.14; collision box size=0.07 0.038 0.15
- link utorso: geometry collision box size=0.2 0.25 0.01; collision box size=0.456306 0.341719 0.12
Joints:
- joint back_bkx: limit lower=-0.523599 upper=0.523599 effort=163 velocity=12 -> lower=-0.523599 upper=0.523599 effort=300 velocity=12
- joint back_bky: limit lower=-0.219388 upper=0.538783 effort=245 velocity=9 -> lower=-0.219388 upper=0.538783 effort=445 velocity=9
- joint back_bkz: limit lower=-0.663225 upper=0.663225 effort=62 velocity=12 -> lower=-0.663225 upper=0.663225 effort=106 velocity=12
- joint l_arm_elx: limit lower=0 upper=2.35619 effort=159 velocity=12 -> lower=0 upper=2.35619 effort=112 velocity=12
- joint l_arm_ely: limit lower=0 upper=3.14159 effort=106 velocity=12 -> lower=0 upper=3.14159 effort=63 velocity=12; origin xyz=0 0.187 0.016 rpy=0 -0 0 -> xyz=0 0.187 -0.016 rpy=0 -0 0
- joint l_arm_shx: limit lower=-1.5708 upper=1.5708 effort=159 velocity=12 -> lower=-1.5708 upper=1.5708 effort=99 velocity=12; origin xyz=0 0.0981 -0.2511 rpy=0 -0 0 -> xyz=0 0.11 -0.245 rpy=0 -0 0
- joint l_arm_shz: limit lower=-1.5708 upper=0.785398 effort=198 velocity=12 -> lower=-1.5708 upper=0.785398 effort=87 velocity=12; origin xyz=0.1406 0.2036 0.4776 rpy=0 -0 0 -> xyz=0.1406 0.2256 0.4776 rpy=0 -0 0
- joint l_arm_wrx: limit lower=-1.1781 upper=1.1781 effort=56 velocity=12 -> lower=-1.1781 upper=1.1781 effort=25 velocity=12; parent l_farm -> l_ufarm
- joint l_arm_wry: child l_farm -> l_ufarm; limit lower=0 upper=3.14159 effort=106 velocity=12 -> lower=0 upper=3.14159 effort=25 velocity=12
- joint l_leg_akx: limit lower=-0.8 upper=0.8 effort=45 velocity=12 -> lower=-0.8 upper=0.8 effort=360 velocity=12
- joint l_leg_aky: limit lower=-1 upper=0.7 effort=350 velocity=12 -> lower=-1 upper=0.7 effort=740 velocity=12
- joint l_leg_hpx: limit lower=-0.523599 upper=0.523599 effort=257 velocity=12 -> lower=-0.523599 upper=0.523599 effort=530 velocity=12
- joint l_leg_hpy: limit lower=-1.61234 upper=0.65764 effort=400 velocity=12 -> lower=-1.61234 upper=0.65764 effort=840 velocity=12
- joint l_leg_hpz: limit lower=-0.174358 upper=0.786794 effort=150 velocity=12 -> lower=-0.174358 upper=0.786794 effort=275 velocity=12
- joint l_leg_kny: limit lower=0 upper=2.35637 effort=246 velocity=12 -> lower=0 upper=2.35637 effort=890 velocity=12
- joint r_arm_elx: limit lower=-2.35619 upper=0 effort=159 velocity=12 -> lower=-2.35619 upper=0 effort=112 velocity=12
- joint r_arm_ely: limit lower=0 upper=3.14159 effort=106 velocity=12 -> lower=0 upper=3.14159 effort=63 velocity=12; origin xyz=0 -0.187 0.016 rpy=0 -0 0 -> xyz=0 -0.187 -0.016 rpy=0 -0 0
- joint r_arm_shx: limit lower=-1.5708 upper=1.5708 effort=159 velocity=12 -> lower=-1.5708 upper=1.5708 effort=99 velocity=12; origin xyz=0 -0.0981 -0.2511 rpy=0 -0 0 -> xyz=0 -0.11 -0.245 rpy=0 -0 0
- joint r_arm_shz: limit lower=-0.785398 upper=1.5708 effort=198 velocity=12 -> lower=-0.785398 upper=1.5708 effort=87 velocity=12; origin xyz=0.1406 -0.2036 0.4776 rpy=0 -0 0 -> xyz=0.1406 -0.2256 0.4776 rpy=0 -0 0
- joint r_arm_wrx: limit lower=-1.1781 upper=1.1781 effort=56 velocity=12 -> lower=-1.1781 upper=1.1781 effort=25 velocity=12; parent r_farm -> r_ufarm
- joint r_arm_wry: child r_farm -> r_ufarm; limit lower=0 upper=3.14159 effort=106 velocity=12 -> lower=0 upper=3.14159 effort=25 velocity=12
- joint r_leg_akx: limit lower=-0.8 upper=0.8 effort=45 velocity=12 -> lower=-0.8 upper=0.8 effort=360 velocity=12
- joint r_leg_aky: limit lower=-1 upper=0.7 effort=350 velocity=12 -> lower=-1 upper=0.7 effort=740 velocity=12
- joint r_leg_hpx: limit lower=-0.523599 upper=0.523599 effort=257 velocity=12 -> lower=-0.523599 upper=0.523599 effort=530 velocity=12
- joint r_leg_hpy: limit lower=-1.61234 upper=0.65764 effort=400 velocity=12 -> lower=-1.61234 upper=0.65764 effort=840 velocity=12
- joint r_leg_hpz: limit lower=-0.786794 upper=0.174358 effort=150 velocity=12 -> lower=-0.786794 upper=0.174358 effort=275 velocity=12
- joint r_leg_kny: limit lower=0 upper=2.35637 effort=246 velocity=12 -> lower=0 upper=2.35637 effort=890 velocity=12
