Commit message: Fixed the .urdf model. See issue #30.

File: ihmc_models/urdf/atlas_unplugged_v5_no_hands.urdf (robot description, URDF)
Before this commit: robot drc_skeleton, 35 links, 34 joints
Links:
- added link center_bottom_led_frame, mass 1e-5
- added link center_top_led_frame, mass 1e-5
- added link head_hokuyo_frame, mass 1e-5
- added link head_imu_link, mass 1e-5; visual box size=0.01 0.01 0.01
- added link hokuyo_link, mass 0.057654; collision box size=0.08 0.06 0.04238; collision cylinder length=0.047 radius=0.024425
- added link imu_link, mass 0.1; visual box size=0.01 0.01 0.01
- added link left_camera_frame, mass 1e-5
- added link left_camera_optical_frame
- added link left_led_frame, mass 1e-5
- added link right_camera_frame, mass 1e-5
- added link right_camera_optical_frame
- added link right_led_frame, mass 1e-5
- link head: mass None -> 1.41984; geometry collision box size=0.0468 0.12 0.1184; collision box size=0.1311 0.12 0.0591
- link l_clav: mass 3.45 -> 4.466
- link l_foot: mass 2.05 -> 2.410
- link l_larm: mass 2.509 -> 3.248
- link l_lglut: mass 0.866 -> 0.898; geometry collision box size=0.0975 0.069 0.103; collision box size=0.125 0.05 0.08
- link l_lleg: mass 5.479 -> 4.515
- link l_scap: mass 3.012 -> 3.899
- link l_uarm: mass 3.388 -> 4.386
- link l_uglut: mass 0.648 -> 1.959; geometry collision box size=0.05 0.1 0.1; collision cylinder length=0.080842 radius=0.019841
- link l_uleg: mass 9.209 -> 8.204
- link ltorso: mass 2.409 -> 2.270
- link mtorso: mass 0.69 -> 0.799
- link pelvis: mass 17.882 -> 9.509
- link r_clav: mass 3.45 -> 4.466
- link r_foot: mass 2.05 -> 2.41
- link r_larm: mass 2.509 -> 3.248
- link r_lglut: mass 0.866 -> 0.898; geometry collision box size=0.0975 0.069 0.103; collision box size=0.125 0.05 0.08
- link r_lleg: mass 5.479 -> 4.515
- link r_scap: mass 3.012 -> 3.899
- link r_uarm: mass 3.388 -> 4.386
- link r_uglut: mass 0.648 -> 1.959; geometry collision box size=0.05 0.1 0.1; collision cylinder length=0.080842 radius=0.019841
- link r_uleg: mass 9.209 -> 8.204
- link utorso: mass 63.73 -> 84.409; geometry collision box size=0.13 0.50 0.10; collision box size=0.2 0.18 0.10
Joints:
- added joint center_bottom_led_frame_joint: type fixed, parent head, child center_bottom_led_frame, origin xyz=0.01125 0.0 -0.0155
- added joint center_top_led_frame_joint: type fixed, parent head, child center_top_led_frame, origin xyz=0.01125 0.0 0.0105
- added joint head_hokuyo_joint: type fixed, parent hokuyo_link, child head_hokuyo_frame, origin xyz=0.03 0 0.015 rpy=0 0 0, axis 0 1 0
- added joint head_imu_joint: type fixed, parent head, child head_imu_link, origin xyz=-0.0475 0.035 0.0 rpy=0 0 0
- added joint hokuyo_joint: type continuous, parent head, child hokuyo_link, origin xyz=-0.0446 0 0.0880 rpy=0 0 0, axis 1 0 0
- added joint imu_joint: type fixed, parent pelvis, child imu_link, origin xyz=0.05991527603 0 -0.01415 rpy=0 0 0
- added joint left_camera_frame_joint: type fixed, parent head, child left_camera_frame, origin xyz=0.0 0.035 -0.002
- added joint left_camera_optical_frame_joint: type fixed, parent left_camera_frame, child left_camera_optical_frame, origin xyz=0 0 0 rpy=-1.5708 0.0 -1.5708
- added joint left_led_frame_joint: type fixed, parent head, child left_led_frame, origin xyz=-0.01443 0.07452 0.050346 rpy=0 -0.15 0.53
- added joint right_camera_frame_joint: type fixed, parent head, child right_camera_frame, origin xyz=0.0 -0.035 -0.002
- added joint right_camera_optical_frame_joint: type fixed, parent right_camera_frame, child right_camera_optical_frame, origin xyz=0 0 0 rpy=-1.5708 0.0 -1.5708
- added joint right_led_frame_joint: type fixed, parent head, child right_led_frame, origin xyz=-0.01443 -0.07452 0.050346 rpy=0 -0.15 -0.53
- joint neck_ry: origin xyz=0.2946 0 0.5765 rpy=0 0 0 -> xyz=0.2546 0 0.6215 rpy=0 0 0

Commit message: Tweaked the .urdf in ihmc_models so it can be used by ihmc_gazebo; the .urdf now more closely matches the model used by the IHMC controller.

File: ihmc_models/urdf/atlas_unplugged_v5_no_hands.urdf (robot description, URDF)
Before this commit: robot atlas, 47 links, 46 joints
Links:
- link l_hand: mass 0.5839 -> 1.7839
- link l_lfarm: mass 0.648 -> 1.6
- link r_hand: mass 0.5839 -> 1.7839
- link r_lfarm: mass 0.648 -> 1.6
Joints:
- joint imu_joint: origin xyz=0.05991527603 0 -0.01415 rpy=0 0 0 -> xyz=-0.0905 -0.000004 -0.0125 rpy=0 3.14159265359 -0.78539816339

Commit message: Reset IMU pose

File: ihmc_models/urdf/atlas_unplugged_v5_no_hands.urdf (robot description, URDF)
Before this commit: robot atlas, 47 links, 46 joints
Joints:
- joint imu_joint: origin xyz=-0.0905 -0.000004 -0.0125 rpy=0 3.14159265359 -0.78539816339 -> xyz=0 0 0 rpy=0 0 0
